File: SPE-Converter.kicad_pcb (KiCad board)
At the start: 4 copper layers, 82 x 56 mm, 199 parts, among them CN401 1.0T-4P_C145956, CN601 2304372-1, CN701 HC-SFP-20P, CN801 39-30-1020, J501 1149873, J601 2374901-1, Q301 HL3407A, SW902 SMWA-08B-TP, U201 DP83TC812RRHARQ1, U301 DP83869HMRGZR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

Commit message: finially done
Parts:
- added C506: 1n 2kV X7R, Capacitor_SMD:C_1210_3225Metric, F.Cu at (58.5, 54.8)
- added C508: 1n 2kV X7R, Capacitor_SMD:C_1210_3225Metric, F.Cu at (73.0, 85.1)
- added H102: JLC_Tooling_Hole, project:JLC_Tooling_Hole, F.Cu at (130.0, 52.0)
- added H103: JLC_Tooling_Hole, project:JLC_Tooling_Hole, F.Cu at (52.0, 52.0)
- added H104: JLC_Tooling_Hole, project:JLC_Tooling_Hole, F.Cu at (52.5, 96.5)
- added R508: 1M, Resistor_SMD:R_1206_3216Metric, F.Cu at (121.8, 80.3)
- added R509: 1M, Resistor_SMD:R_1206_3216Metric, F.Cu at (73.0, 80.5)
- C507, R506: moved to F.Cu
- J501: footprint SamacSys_Parts:1149873 -> project:1149873
- J601: footprint SamacSys_Parts:23749011 -> project:23749011
- moved C507 53.8 mm to (124.5, 80.3)
- moved R506 36.7 mm to (58.5, 52.0), turned to 0 degrees
- moved C501 3.30 mm to (73.6, 86.5), turned to 180 degrees
- moved J601 0.16 mm to (118.7, 91.6)
Connections:
- U701 pad 10: Earth -> unconnected-(U701-Pad10)
- U701 pad 11: Earth -> unconnected-(U701-Pad11)
- U701 pad 12: Earth -> unconnected-(U701-Pad12)
- U701 pad 13: Earth -> unconnected-(U701-Pad13)
- U701 pad 14: Earth -> unconnected-(U701-Pad14)
- U701 pad 15: Earth -> unconnected-(U701-Pad15)
- U701 pad 19: Earth -> unconnected-(U701-Pad19)
- U701 pad 8: Earth -> unconnected-(U701-Pad8)
- U701 pad 9: Earth -> unconnected-(U701-Pad9)
Routing:
- net GND: track 148.9 -> 154.1 mm, vias 121 -> 188
- net +3.3V: track 75.4 -> 79.6 mm
- net Earth: track 0.00 -> 2.87 mm, vias 0 -> 3
- net Net-(C501-Pad1): track 12.3 -> 14.7 mm
- net /MSP M0/RGB_BLUE: track 27.2 -> 25.8 mm
- net /MSP M0/RGB_RED: track 26.1 -> 24.8 mm
- net /SPE PHY/AUTO_STRAP: track 34.2 -> 35.3 mm
- net (no net): vias 1 -> 0
- added copper zone on B.Cu, net Earth
- added copper zone on F.Cu, net Earth
Other:
- board text added: "+ -"
- board text added: "12V supply"
- board text added: "Designed by Matteo Valentini"
- board text added: "github.com/vl9i/spe-converter"
