File: rj45.kicad_sch (KiCad schematic)
At the start: 17 parts, among them J501 1149873

Commit message: finially done
Parts:
- added C506, C508: 1n 2kV X7R, Capacitor_SMD:C_1210_3225Metric, symbol Device:C_Small
- added R508, R509: 1M, Resistor_SMD:R_1206_3216Metric, symbol Device:R_Small
- J501: footprint 1149873 -> project:1149873; symbol SamacSys_Parts:1149873 -> project:1149873
Connections:
- net Earth: now also C506.2, C508.2, R508.1, R509.1
- net GND: now also C506.1, C508.1, R508.2, R509.2
