File: sfp.kicad_sch (KiCad schematic)
At the start: 20 parts, among them CN701 HC-SFP-20P, U701 HC-SFP-01L

Commit message: finially done
Connections:
- net Earth: no longer U701.10, U701.11, U701.12, U701.13, U701.14, U701.15, U701.19, U701.8, U701.9
- no-connect marks 0 -> 9
Changed lines of the file:
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@@
-	)
-	(junction
-		(at 144.78 148.59)
-		(diameter 0)
-		(color 0 0 0 0)
 	)
 	(junction
@@
 	)
 	(junction
-		(at 124.46 151.13)
+		(at 144.78 143.51)
 		(diameter 0)
 		(color 0 0 0 0)
@@
 	)
 	(junction
-		(at 144.78 151.13)
-		(diameter 0)
-		(color 0 0 0 0)
-	)
-	(junction
 		(at 154.94 52.07)
 		(diameter 0)
@@
 	)
 	(junction
-		(at 144.78 153.67)
-		(diameter 0)
-		(color 0 0 0 0)
-	)
-	(junction
-		(at 124.46 156.21)
-		(diameter 0)
-		(color 0 0 0 0)
-	)
-	(junction
 		(at 124.46 138.43)
 		(diameter 0)
@@
 	)
 	(junction
-		(at 144.78 135.89)
-		(diameter 0)
-		(color 0 0 0 0)
-	)
-	(junction
 		(at 38.1 83.82)
 		(diameter 0)
@@
 	)
 	(junction
-		(at 144.78 146.05)
-		(diameter 0)
-		(color 0 0 0 0)
-	)
-	(junction
 		(at 85.09 85.09)
 		(diameter 0)
@@
 	)
 	(junction
-		(at 144.78 143.51)
-		(diameter 0)
-		(color 0 0 0 0)
-	)
-	(junction
 		(at 231.14 95.25)
 		(diameter 0)
@@
 	)
 	(junction
-		(at 124.46 153.67)
-		(diameter 0)
-		(color 0 0 0 0)
-	)
-	(junction
-		(at 144.78 156.21)
-		(diameter 0)
-		(color 0 0 0 0)
-	)
-	(junction
 		(at 124.46 135.89)
 		(diameter 0)
 		(color 0 0 0 0)
+	)
+	(no_connect
+		(at 127 153.67)
+	)
+	(no_connect
+		(at 142.24 135.89)
+	)
+	(no_connect
+		(at 127 156.21)
+	)
+	(no_connect
+		(at 142.24 156.21)
+	)
+	(no_connect
+		(at 127 151.13)
+	)
+	(no_connect
+		(at 142.24 153.67)
+	)
+	(no_connect
+		(at 142.24 146.05)
+	)
+	(no_connect
+		(at 142.24 148.59)
+	)
+	(no_connect
+		(at 142.24 151.13)
 	)
 	(bus_entry
@@
 	(wire
 		(pts
-			(xy 124.46 151.13) (xy 127 151.13)
-		)
-		(stroke
-			(width 0)
-			(type default)
-		)
-	)
-	(wire
-		(pts
 			(xy 64.77 83.82) (xy 64.77 85.09)
 		)
@@
 	(wire
 		(pts
-			(xy 124.46 153.67) (xy 124.46 151.13)
-		)
-		(stroke
-			(width 0)
-			(type default)
-		)
-	)
-	(wire
-		(pts
 			(xy 142.24 92.71) (xy 205.74 92.71)
 		)
@@
 	(wire
 		(pts
-			(xy 124.46 158.75) (xy 124.46 156.21)
-		)
-		(stroke
-			(width 0)
-			(type default)
-		)
-	)
-	(wire
-		(pts
 			(xy 64.77 85.09) (xy 85.09 85.09)
 		)
@@
 	(wire
 		(pts
-			(xy 142.24 148.59) (xy 144.78 148.59)
-		)
-		(stroke
-			(width 0)
-			(type default)
-		)
-	)
-	(wire
-		(pts
 			(xy 177.8 58.42) (xy 177.8 82.55)
 		)
@@
 	(wire
 		(pts
-			(xy 124.46 153.67) (xy 127 153.67)
-		)
-		(stroke
-			(width 0)
-			(type default)
-		)
-	)
-	(wire
-		(pts
 			(xy 154.94 52.07) (xy 177.8 52.07)
 		)
@@
 	(wire
 		(pts
-			(xy 124.46 151.13) (xy 124.46 148.59)
+			(xy 124.46 148.59) (xy 124.46 158.75)
 		)
 		(stroke
@@
 	(wire
 		(pts
-			(xy 142.24 135.89) (xy 144.78 135.89)
-		)
-		(stroke
-			(width 0)
-			(type default)
-		)
-	)
-	(wire
-		(pts
 			(xy 142.24 95.25) (xy 231.14 95.25)
 		)
@@
 	(wire
 		(pts
-			(xy 144.78 135.89) (xy 144.78 138.43)
+			(xy 144.78 133.35) (xy 144.78 138.43)
 		)
 		(stroke
@@
 	(wire
 		(pts
-			(xy 142.24 153.67) (xy 144.78 153.67)
-		)
-		(stroke
-			(width 0)
-			(type default)
-		)
-	)
-	(wire
-		(pts
 			(xy 142.24 133.35) (xy 144.78 133.35)
 		)
@@
 	(wire
 		(pts
-			(xy 144.78 156.21) (xy 144.78 158.75)
-		)
-		(stroke
-			(width 0)
-			(type default)
-		)
-	)
-	(wire
-		(pts
-			(xy 142.24 156.21) (xy 144.78 156.21)
-		)
-		(stroke
-			(width 0)
-			(type default)
-		)
-	)
-	(wire
-		(pts
-			(xy 124.46 156.21) (xy 127 156.21)
-		)
-		(stroke
-			(width 0)
-			(type default)
-		)
-	)
-	(wire
-		(pts
 			(xy 203.2 52.07) (xy 205.74 52.07)
 		)
@@
 	(wire
 		(pts
-			(xy 144.78 133.35) (xy 144.78 135.89)
-		)
-		(stroke
-			(width 0)
-			(type default)
-		)
-	)
-	(wire
-		(pts
 			(xy 180.34 52.07) (xy 184.15 52.07)
 		)
@@
 	(wire
 		(pts
-			(xy 142.24 146.05) (xy 144.78 146.05)
-		)
-		(stroke
-			(width 0)
-			(type default)
-		)
-	)
-	(wire
-		(pts
 			(xy 152.4 58.42) (xy 152.4 77.47)
 		)
@@
 	(wire
 		(pts
+			(xy 144.78 143.51) (xy 144.78 158.75)
+		)
+		(stroke
+			(width 0)
+			(type default)
+		)
+	)
+	(wire
+		(pts
 			(xy 107.95 80.01) (xy 127 80.01)
 		)
@@
 	(wire
 		(pts
-			(xy 144.78 143.51) (xy 144.78 146.05)
-		)
-		(stroke
-			(width 0)
-			(type default)
-		)
-	)
-	(wire
-		(pts
-			(xy 144.78 153.67) (xy 144.78 156.21)
-		)
-		(stroke
-			(width 0)
-			(type default)
-		)
-	)
-	(wire
-		(pts
 			(xy 152.4 77.47) (xy 234.95 77.47)
 		)
@@
 	(wire
 		(pts
-			(xy 144.78 148.59) (xy 144.78 151.13)
-		)
-		(stroke
-			(width 0)
-			(type default)
-		)
-	)
-	(wire
-		(pts
 			(xy 142.24 140.97) (xy 144.78 140.97)
 		)
@@
 	(wire
 		(pts
-			(xy 144.78 146.05) (xy 144.78 148.59)
-		)
-		(stroke
-			(width 0)
-			(type default)
-		)
-	)
-	(wire
-		(pts
 			(xy 64.77 87.63) (xy 85.09 87.63)
 		)
@@
 	(wire
 		(pts
-			(xy 124.46 156.21) (xy 124.46 153.67)
-		)
-		(stroke
-			(width 0)
-			(type default)
-		)
-	)
-	(wire
-		(pts
 			(xy 154.94 58.42) (xy 154.94 80.01)
 		)
@@
 	(wire
 		(pts
-			(xy 142.24 151.13) (xy 144.78 151.13)
-		)
-		(stroke
-			(width 0)
-			(type default)
-		)
-	)
-	(wire
-		(pts
 			(xy 107.95 102.87) (xy 205.74 102.87)
 		)
@@
 		)
 		(stroke
-			(width 0)
-			(type default)
-		)
-	)
-	(wire
-		(pts
-			(xy 144.78 151.13) (xy 144.78 153.67)
-		)
-		(stroke
