File: spe_conn.kicad_sch (KiCad schematic)
At the start: 22 parts, among them CN601 2304372-1, J601 2374901-1, U601 TMUX136RSER

Commit message: finially done
Parts:
- J601: footprint 23749011 -> project:23749011; symbol SamacSys_Parts:2374901-1 -> project:2374901-1
Changed lines of the file:
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@@
 	)
 	(symbol
-		(lib_id "SamacSys_Parts:2374901-1")
+		(lib_id "project:2374901-1")
 		(at 62.23 101.6 0)
 		(mirror y)
@@
 			)
 		)
-		(property "Footprint" "23749011"
+		(property "Footprint" "project:23749011"
 			(at 40.64 196.52 0)
 			(hide yes)
